File: Core v2/Core v2.kicad_pcb (KiCad board)
At the start: 4 copper layers, 44.3 x 56 mm, 92 parts, among them CN1 PJ-3200, J1 Serial Debug, J2 USB_C_Receptacle_USB2.0, Q1 BSS138, SW1 SW_SPST, SW2 SW_SPST, SW3 SW_SPST, U1 DL-TX1-433M, U2 H34B-433M, U3 ESP32-S3-WROOM-1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

Commit message: Core V2.1 KiCad + JLC Files
Parts:
- removed kibuzzard-658A2FFC: G***, kibuzzard-658A2FFC
- removed kibuzzard-658A3003: G***, kibuzzard-658A3003
- removed kibuzzard-658A3009: G***, kibuzzard-658A3009
- removed kibuzzard-658A3013: G***, kibuzzard-658A3013
- removed kibuzzard-65AF1A0B: G***, kibuzzard-65AF1A0B
- removed kibuzzard-65AF1A15: G***, kibuzzard-65AF1A15
- added C13: 100nF, Capacitor_SMD:C_0603_1608Metric_Pad1.08x0.95mm_HandSolder, F.Cu at (112.8, 101.2)
- added L1: L, Inductor_SMD:L_0603_1608Metric_Pad1.05x0.95mm_HandSolder, F.Cu at (110.2, 70.5)
- added L2: L, Inductor_SMD:L_0603_1608Metric_Pad1.05x0.95mm_HandSolder, F.Cu at (115.2, 70.5)
- added kibuzzard-658A429F: G***, kibuzzard-658A429F, F.Cu at (118.3, 64.4)
- added kibuzzard-658A42A3: G***, kibuzzard-658A42A3, F.Cu at (118.3, 61.8)
- added kibuzzard-658A42A8: G***, kibuzzard-658A42A8, F.Cu at (118.3, 59.2)
- added kibuzzard-658A42AC: G***, kibuzzard-658A42AC, F.Cu at (118.3, 66.9)
- added kibuzzard-65FD518D: G***, kibuzzard-65FD518D, B.Cu at (120.0, 59.6)
- added kibuzzard-65FD5191: G***, kibuzzard-65FD5191, B.Cu at (119.9, 66.0)
- AE1: footprint Connector_PinHeader_2.54mm:PinHeader_1x01_P2.54mm_Vertical -> Connector_Pin:Pin_D1.0mm_L10.0mm
- REF**: moved to F.Cu
- moved kibuzzard-658A429F 16.6 mm to (112.0, 59.2), turned to -90 degrees
- moved REF** 16.6 mm to (105.2, 76.6)
- moved kibuzzard-658A42A3 13.7 mm to (112.0, 61.8), turned to -90 degrees
- moved kibuzzard-658A42AC 13.1 mm to (112.0, 67.0), turned to -90 degrees
- moved kibuzzard-658A42A8 12.4 mm to (112.0, 64.3), turned to -90 degrees
- moved C12 11.4 mm to (112.7, 69.6)
- moved U1 9.63 mm to (113.6, 63.1), turned to 0 degrees
- moved AE1 6.16 mm to (104.5, 58.5), turned to -90 degrees
- moved JP1 5.83 mm to (119.9, 63.0), turned to -90 degrees
- moved R4 5.28 mm to (136.4, 66.2), turned to -90 degrees
- moved U2 4.89 mm to (116.5, 63.1), turned to 90 degrees
- moved kibuzzard-658A25BD 4.23 mm to (118.5, 63.0), turned to -90 degrees
- moved REF** 3.50 mm to (105.1, 68.0), turned to 90 degrees
- moved C5 3.43 mm to (111.0, 106.2)
- moved C7 2.62 mm to (114.0, 108.2), turned to -90 degrees
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Connections:
- JP1 pad 1: +5V -> +3V3
- JP1 pad 3: +3V3 -> +5V
Routing:
- net GND: track 39.2 -> 20.6 mm, vias 53 -> 59
- net +3V3: track 117.7 -> 99.3 mm, vias 7 -> 6
- net Net-(AE1-A): track 5.36 -> 18.0 mm
- net RF_Power: track 23.7 -> 32.5 mm
- net RF_Shifted: track 18.9 -> 24.4 mm
- net E_STOP: track 38.5 -> 42.1 mm
- net EN: track 69.2 -> 72.8 mm
- net Net-(U1-ANT): track 9.49 -> 7.42 mm
- net +5V: track 29.5 -> 28.2 mm, vias 4 -> 3
- net CC1: track 7.65 -> 8.15 mm
Other:
- board text added: "1"
- board text removed: "0"

Commit message: Core V2.2 KiCad + JLC Files
Parts:
- U5: value AMS1117-3.3 -> AP2114HA-3.3
- moved TP1 1.10 mm to (121.5, 94.5)
- moved TP2 1.10 mm to (119.2, 94.5)
- moved TP3 1.10 mm to (116.8, 94.5)
- moved TP4 1.10 mm to (114.4, 94.5)
- moved TP5 1.10 mm to (126.3, 94.5)
- moved TP6 1.10 mm to (123.9, 94.5)
- moved C10 0.62 mm to (118.1, 77.9)
- moved C13 0.20 mm to (112.8, 101.4)
- moved FID1 0.05 mm to (100.7, 57.7)
- moved FID4 0.05 mm to (100.7, 111.8)
- turned AE1 to 90 degrees
Connections:
- U5 pad 1: GND -> +5V
- U5 pad 2: +3V3 -> GND
- U5 pad 3: +5V -> +3V3
Routing:
- net +5V: track 28.2 -> 75.2 mm, vias 3 -> 4
- net +3V3: track 99.3 -> 141.6 mm, vias 6 -> 7
- net GND: track 20.6 -> 35.9 mm, vias 59 -> 85
- net +5VA: track 15.4 -> 28.5 mm
- net EN: track 72.8 -> 77.2 mm
- net MTDO: track 15.1 -> 14.0 mm
- net MTDI: track 14.9 -> 13.8 mm
- net MTCK: track 15.1 -> 14.0 mm
- net MTMS: track 16.1 -> 15.3 mm
- net RGB: track 13.4 -> 13.9 mm
- removed copper zone on In2.Cu, net +3V3
- removed copper zone on In2.Cu, net +5V
- removed copper zone on In1.Cu, net GND
- removed copper zone on In2.Cu, net GND
Other:
- outline, holes or cut-outs redrawn
- copper layers 4 -> 2
- board text added: "2"
- board text added: "L"
- board text removed: "1"
